File: InitialDesign/Controller.sch (KiCad schematic (older format))
At the start: 11 parts, among them J5 Conn_01x02, J6 Conn_01x02, U2 STM32F042C6T6

Commit message: Schematic and Layout commenced
Parts:
- C3, C4, C5, C6, C7, C8, C9: footprint (none) -> Capacitors_SMD:C_0805
- J5, J6: footprint (none) -> Pin_Headers:Pin_Header_Straight_1x02_Pitch2.54mm
- R5: footprint (none) -> Resistors_SMD:R_0805
- U2: footprint Housings_DFN_LQFP:LQFP-48-1EP_7x7mm_Pitch0.5mm -> Housings_QFP:LQFP-48_7x7mm_Pitch0.5mm
Changed lines of the file:
@@
 F 0 "U2" H 3500 5900 50  0000 C CNN
 F 1 "STM32F042C6T6" H 7450 1900 50  0000 C CNN
-F 2 "Housings_DFN_LQFP:LQFP-48-1EP_7x7mm_Pitch0.5mm" H 5400 1850 50  0001 C CIN
+F 2 "Housings_QFP:LQFP-48_7x7mm_Pitch0.5mm" H 5400 1850 50  0001 C CIN
 F 3 "" H 5600 4100 50  0000 C CNN
 	1    5600 3850
@@
 LED2_GREEN
 $Comp
-L GND #PWR016
+L GND #PWR018
 U 1 1 5A520153
 P 3100 5800
-F 0 "#PWR016" H 3100 5550 50  0001 C CNN
+F 0 "#PWR018" H 3100 5550 50  0001 C CNN
 F 1 "GND" H 3100 5650 50  0000 C CNN
 F 2 "" H 3100 5800 50  0001 C CNN
@@
 F 0 "C3" H 925 1600 50  0000 L CNN
 F 1 "10nF" H 925 1400 50  0000 L CNN
-F 2 "" H 938 1350 50  0001 C CNN
+F 2 "Capacitors_SMD:C_0805" H 938 1350 50  0001 C CNN
 F 3 "" H 900 1500 50  0001 C CNN
 	1    900  1500
@@
 F 0 "C6" H 1225 1600 50  0000 L CNN
 F 1 "1uF" H 1225 1400 50  0000 L CNN
-F 2 "" H 1238 1350 50  0001 C CNN
+F 2 "Capacitors_SMD:C_0805" H 1238 1350 50  0001 C CNN
 F 3 "" H 1200 1500 50  0001 C CNN
 	1    1200 1500
@@
 F 0 "C4" H 925 2300 50  0000 L CNN
 F 1 "100nF" H 925 2100 50  0000 L CNN
-F 2 "" H 938 2050 50  0001 C CNN
+F 2 "Capacitors_SMD:C_0805" H 938 2050 50  0001 C CNN
 F 3 "" H 900 2200 50  0001 C CNN
 	1    900  2200
@@
 F 0 "C7" H 1225 2300 50  0000 L CNN
 F 1 "100nF" H 1225 2100 50  0000 L CNN
-F 2 "" H 1238 2050 50  0001 C CNN
+F 2 "Capacitors_SMD:C_0805" H 1238 2050 50  0001 C CNN
 F 3 "" H 1200 2200 50  0001 C CNN
 	1    1200 2200
@@
 F 0 "C9" H 1525 2300 50  0000 L CNN
 F 1 "4.7uF" H 1525 2100 50  0000 L CNN
-F 2 "" H 1538 2050 50  0001 C CNN
+F 2 "Capacitors_SMD:C_0805" H 1538 2050 50  0001 C CNN
 F 3 "" H 1500 2200 50  0001 C CNN
 	1    1500 2200
@@
 F 0 "C5" H 925 3100 50  0000 L CNN
 F 1 "100nF" H 925 2900 50  0000 L CNN
-F 2 "" H 938 2850 50  0001 C CNN
+F 2 "Capacitors_SMD:C_0805" H 938 2850 50  0001 C CNN
 F 3 "" H 900 3000 50  0001 C CNN
 	1    900  3000
@@
 F 0 "C8" H 1225 3100 50  0000 L CNN
 F 1 "4.7uF" H 1225 2900 50  0000 L CNN
-F 2 "" H 1238 2850 50  0001 C CNN
+F 2 "Capacitors_SMD:C_0805" H 1238 2850 50  0001 C CNN
 F 3 "" H 1200 3000 50  0001 C CNN
 	1    1200 3000
@@
 	900  2850 1500 2850
 $Comp
-L GND #PWR017
+L GND #PWR019
 U 1 1 5A521823
 P 900 1650
-F 0 "#PWR017" H 900 1400 50  0001 C CNN
+F 0 "#PWR019" H 900 1400 50  0001 C CNN
 F 1 "GND" H 900 1500 50  0000 C CNN
 F 2 "" H 900 1650 50  0001 C CNN
@@
 $EndComp
 $Comp
-L GND #PWR018
+L GND #PWR020
 U 1 1 5A521849
 P 900 2350
-F 0 "#PWR018" H 900 2100 50  0001 C CNN
+F 0 "#PWR020" H 900 2100 50  0001 C CNN
 F 1 "GND" H 900 2200 50  0000 C CNN
 F 2 "" H 900 2350 50  0001 C CNN
@@
 $EndComp
 $Comp
-L GND #PWR019
+L GND #PWR021
 U 1 1 5A52186F
 P 900 3150
-F 0 "#PWR019" H 900 2900 50  0001 C CNN
+F 0 "#PWR021" H 900 2900 50  0001 C CNN
 F 1 "GND" H 900 3000 50  0000 C CNN
 F 2 "" H 900 3150 50  0001 C CNN
@@
 Connection ~ 1200 2350
 $Comp
-L +3V3 #PWR020
+L +3V3 #PWR022
 U 1 1 5A521918
 P 3050 1800
-F 0 "#PWR020" H 3050 1650 50  0001 C CNN
+F 0 "#PWR022" H 3050 1650 50  0001 C CNN
 F 1 "+3V3" H 3050 1940 50  0000 C CNN
 F 2 "" H 3050 1800 50  0001 C CNN
@@
 	3050 1950 3050 1800
 $Comp
-L +3V3 #PWR021
+L +3V3 #PWR023
 U 1 1 5A521964
 P 900 1350
-F 0 "#PWR021" H 900 1200 50  0001 C CNN
+F 0 "#PWR023" H 900 1200 50  0001 C CNN
 F 1 "+3V3" H 900 1490 50  0000 C CNN
 F 2 "" H 900 1350 50  0001 C CNN
@@
 $EndComp
 $Comp
-L +3V3 #PWR022
+L +3V3 #PWR024
 U 1 1 5A521988
 P 900 2050
-F 0 "#PWR022" H 900 1900 50  0001 C CNN
+F 0 "#PWR024" H 900 1900 50  0001 C CNN
 F 1 "+3V3" H 900 2190 50  0000 C CNN
 F 2 "" H 900 2050 50  0001 C CNN
@@
 $EndComp
 $Comp
-L +3V3 #PWR023
+L +3V3 #PWR025
 U 1 1 5A5219D6
 P 900 2850
-F 0 "#PWR023" H 900 2700 50  0001 C CNN
+F 0 "#PWR025" H 900 2700 50  0001 C CNN
 F 1 "+3V3" H 900 2990 50  0000 C CNN
 F 2 "" H 900 2850 50  0001 C CNN
@@
 F 0 "R5" V 1130 4100 50  0000 C CNN
 F 1 "10k" V 1050 4100 50  0000 C CNN
-F 2 "" V 980 4100 50  0001 C CNN
+F 2 "Resistors_SMD:R_0805" V 980 4100 50  0001 C CNN
 F 3 "" H 1050 4100 50  0001 C CNN
 	1    1050 4100
@@
 F 0 "J5" H 950 3750 50  0000 C CNN
 F 1 "Conn_01x02" V 1050 3650 50  0000 C CNN
-F 2 "" H 950 3650 50  0001 C CNN
+F 2 "Pin_Headers:Pin_Header_Straight_1x02_Pitch2.54mm" H 950 3650 50  0001 C CNN
 F 3 "" H 950 3650 50  0001 C CNN
 	1    950  3650
@@
 Connection ~ 1050 3900
 $Comp
-L +3V3 #PWR024
+L +3V3 #PWR026
 U 1 1 5A52C7B4
 P 750 3950
-F 0 "#PWR024" H 750 3800 50  0001 C CNN
+F 0 "#PWR026" H 750 3800 50  0001 C CNN
 F 1 "+3V3" H 750 4090 50  0000 C CNN
 F 2 "" H 750 3950 50  0001 C CNN
@@
 	750  4050 750  3950
 $Comp
-L GND #PWR025
+L GND #PWR027
 U 1 1 5A52C800
 P 1050 4250
-F 0 "#PWR025" H 1050 4000 50  0001 C CNN
+F 0 "#PWR027" H 1050 4000 50  0001 C CNN
 F 1 "GND" H 1050 4100 50  0000 C CNN
 F 2 "" H 1050 4250 50  0001 C CNN
@@
 F 0 "J6" H 950 4800 50  0000 C CNN
 F 1 "Conn_01x02" V 1050 4700 50  0000 C CNN
-F 2 "" H 950 4700 50  0001 C CNN
+F 2 "Pin_Headers:Pin_Header_Straight_1x02_Pitch2.54mm" H 950 4700 50  0001 C CNN
 F 3 "" H 950 4700 50  0001 C CNN
 	1    950  4700
@@
 $EndComp
 $Comp
-L GND #PWR026
+L GND #PWR028
 U 1 1 5A52D66B
 P 950 4900
-F 0 "#PWR026" H 950 4650 50  0001 C CNN
+F 0 "#PWR028" H 950 4650 50  0001 C CNN
 F 1 "GND" H 950 4750 50  0000 C CNN
 F 2 "" H 950 4900 50  0001 C CNN
