File: InitialDesign/InitialDesign.kicad_pcb (KiCad board)
At the start: 2 copper layers, 122.5 x 115.6 mm, 44 parts, among them J1 Conn_01x07_Female, J2 Conn_01x04, J3 Conn_01x04, J4 USB_OTG, J5 Conn_01x02, J6 Conn_01x02, J7 Conn_02x15_Odd_Even, U1 TPS61222DCKR, U2 STM32F042C6T6, U3 M24SR02-YMN6T

Commit message: Initial proto done
Parts:
- added FID1: Fiducial, Fiducials:Fiducial_1.5mm_Dia_2.54mm_Outer_CopperTop, F.Cu at (106.8, 156.3)
- added FID2: Fiducial, Fiducials:Fiducial_1.5mm_Dia_2.54mm_Outer_CopperTop, F.Cu at (202.2, 96.6)
- added FID3: Fiducial, Fiducials:Fiducial_1.5mm_Dia_2.54mm_Outer_CopperTop, F.Cu at (136.4, 52.4)
- added J8: Conn_02x02_Odd_Even, Pin_Headers:Pin_Header_Straight_2x02_Pitch2.54mm, F.Cu at (163.7, 88.9)
- added J9: Conn_02x08_Odd_Even, Pin_Headers:Pin_Header_Straight_2x08_Pitch2.54mm, F.Cu at (141.7, 132.4)
- J7: value Conn_02x15_Odd_Even -> Conn_02x03_Odd_Even; footprint Pin_Headers:Pin_Header_Straight_2x15_Pitch2.54mm -> Pin_Headers:Pin_Header_Straight_2x03_Pitch2.54mm
- moved J7 65.2 mm to (169.1, 113.8), turned to 0 degrees
- moved R6 6.91 mm to (139.1, 121.6)
- moved C9 4.04 mm to (157.6, 125.6), turned to 0 degrees
- moved C7 1.52 mm to (157.6, 124.0), turned to 0 degrees
Connections:
- J7 pad 1: PB4 -> GND
- J7 pad 2: NFC_GPO -> VDD
- J7 pad 3: SWDIO -> SPI1_NSS
- J7 pad 4: PB5 -> OLED_SCL
- J7 pad 5: USB_D- -> SPI1_MISO
- J7 pad 6: USB_D+ -> OLED_SDA
Routing:
- net GND: track 177.1 -> 565.9 mm, vias 3 -> 15
- net VDD: track 107.8 -> 364.0 mm, vias 2 -> 10
- net OLED_SDA: track 12.6 -> 56.4 mm, vias 1 -> 3
- net OLED_SCL: track 14.6 -> 58.3 mm, vias 1 -> 3
- net PB14: track 52.2 -> 17.0 mm, vias 5 -> 2
- net PB5: track 1.26 -> 35.1 mm, vias 1 -> 2
- net PB12: track 58.4 -> 26.8 mm, vias 5 -> 2
- net LED2_GREEN: track 112.8 -> 81.3 mm, vias 7 -> 4
- net PB4: track 0.00 -> 30.0 mm, vias 0 -> 2
- net NFC_GPO: track 3.55 -> 32.3 mm, vias 1 -> 4
- net SPI1_NSS: track 25.6 -> 54.2 mm
- net USB_D-: track 108.5 -> 83.8 mm
- net NFC_DISABLE: track 13.8 -> 38.2 mm, vias 0 -> 2
- net PB3: track 41.5 -> 25.3 mm
- net PC14: track 11.6 -> 26.3 mm, vias 1 -> 2
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- added copper zone on B.Cu, net VDD
- removed copper zone on F.Cu, net +BATT
- removed copper zone on F.Cu, net Net-(L1-Pad2)
- removed copper zone on F.Cu, net VDD
Other:
- net class Default: clearance 0.2 -> 0.1524
- net class DirtyPCB added: clearance 0.1524, trace_width 0.1524, via_dia 0.6, via_drill 0.4
- rule trace_clearance: 0.2 -> 0.1524
- rule trace_min: 0.1 -> 0.1524
