File: InitialDesign/InitialDesign.sch (KiCad schematic (older format))
At the start: 8 parts, among them J1 Conn_01x07, J2 Conn_01x04, J3 Conn_01x04, J4 USB_A

Commit message: Schematic and Layout commenced
Parts:
- removed J1: Conn_01x07, symbol Conn_01x07
- removed J4: USB_A, symbol USB_A
- added D3, D4, D5, D6, D7: LED, LEDs:LED_1206, symbol LED
- added J1: Conn_01x07_Female, Socket_Strips:Socket_Strip_Straight_1x07_Pitch2.54mm, symbol Conn_01x07_Female
- added J4: USB_OTG, Connectors:USB_Micro-B, symbol USB_OTG
- added J7: Conn_02x15_Odd_Even, Pin_Headers:Pin_Header_Straight_2x15_Pitch2.54mm, symbol Conn_02x15_Odd_Even
- added R10, R11, R7, R8, R9: R, Resistors_SMD:R_0805, symbol R
- D1, D2: footprint (none) -> LEDs:LED_RGB_5050-6
- J2, J3: footprint (none) -> Pin_Headers:Pin_Header_Straight_1x04_Pitch2.54mm
- R1, R2: footprint (none) -> Resistors_SMD:R_0805
Connections:
- net +3V3: now also J1.2 (Pin_2), J4.1 (VBUS), J7.29 (Pin_29)
- net GND: now also D3.1 (K), D4.1 (K), D5.1 (K), D6.1 (K), D7.1 (K), J1.1 (Pin_1), J4.4 (ID), J4.5 (GND), J4.6 (Shield), J7.30 (Pin_30)
- net NFC_GPO: now also J7.2 (Pin_2)
- net NFC_SCL: now also J7.24 (Pin_24)
- net NFC_SDA: now also J7.25 (Pin_25)
- net OLED_BLK: now also J1.7 (Pin_7)
- net OLED_DC_A0: now also J1.6 (Pin_6)
- net OLED_RESET: now also J1.5 (Pin_5)
- net OLED_SCL: now also J1.3 (Pin_3)
- net OLED_SDA: now also J1.4 (Pin_4)
- net SWDIO: now also J7.3 (Pin_3)
- net at R2.1: now also J4.2 (D-)
- net at R1.1: now also J4.3 (D+)
- net Controller/LED1_BLUE renamed LED1_BLUE
- net LED1_BLUE: now also J7.14 (Pin_14)
- net Controller/LED1_GREEN renamed LED1_GREEN
- net LED1_GREEN: now also J7.12 (Pin_12)
- net Controller/LED1_RED renamed LED1_RED
- net LED1_RED: now also J7.7 (Pin_7)
- net Controller/LED2_BLUE renamed LED2_BLUE
- net LED2_BLUE: now also J7.8 (Pin_8)
- net Controller/LED2_GREEN renamed LED2_GREEN
- net LED2_GREEN: now also J7.20 (Pin_20)
- net Controller/LED2_RED renamed LED2_RED
- net LED2_RED: now also J7.10 (Pin_10)
- net Controller/USB_DM renamed USB_D-
- net USB_D-: now also J7.5 (Pin_5)
- net Controller/USB_DP renamed USB_D+
- net USB_D+: now also J7.6 (Pin_6)
- new net: D3.2 (A), R7.1
- new net: D4.2 (A), R8.1
- new net: D5.2 (A), R9.1
- new net: D7.2 (A), R11.1
- new net: D6.2 (A), R10.1
- new net PA0: J7.23 (Pin_23)
- new net PB0: J7.17 (Pin_17)
- new net PB1: J7.22 (Pin_22)
- new net PB11: J7.13 (Pin_13), R7.2
- new net PB12: J7.18 (Pin_18), R8.2
- new net PB13: J7.11 (Pin_11), R9.2
- new net PB14: J7.16 (Pin_16), R10.2
- new net PB15: J7.9 (Pin_9), R11.2
- new net PB3: J7.15 (Pin_15)
- new net PB4: J7.1 (Pin_1)
- new net PB5: J7.4 (Pin_4)
- new net PC13: J7.28 (Pin_28)
- new net PC14: J7.27 (Pin_27)
- new net PC15: J7.26 (Pin_26)
- new net SPI1_MISO: J7.19 (Pin_19)
- new net SPI1_NSS: J7.21 (Pin_21)
- no-connect marks 16 -> 0
Other:
- note added: "Eye LEDs"
- note added: "Teeth LEDs"
- note added: "Test Points"
- moved on the sheet: D1, D2, R1, R2

Commit message: Initial proto done
Parts:
- removed J7: Conn_02x15_Odd_Even, Pin_Headers:Pin_Header_Straight_2x15_Pitch2.54mm, symbol Conn_02x15_Odd_Even
- added FID1, FID2, FID3: Fiducial, Fiducials:Fiducial_1.5mm_Dia_2.54mm_Outer_CopperTop, symbol Fiducial
- added J7: Conn_02x03_Odd_Even, Pin_Headers:Pin_Header_Straight_2x03_Pitch2.54mm, symbol Conn_02x03_Odd_Even
- added J8: Conn_02x02_Odd_Even, Pin_Headers:Pin_Header_Straight_2x02_Pitch2.54mm, symbol Conn_02x02_Odd_Even
- added J9: Conn_02x08_Odd_Even, Pin_Headers:Pin_Header_Straight_2x08_Pitch2.54mm, symbol Conn_02x08_Odd_Even
Connections:
- net +3V3: now also J7.2 (Pin_2), J8.2 (Pin_2), J9.12 (Pin_12), J9.14 (Pin_14), J9.16 (Pin_16), J9.2 (Pin_2)
- net GND: now also J7.1 (Pin_1), J8.1 (Pin_1), J9.1 (Pin_1), J9.13 (Pin_13), J9.15 (Pin_15)
- net NFC_SCL: now also J8.3 (Pin_3)
- net NFC_SDA: now also J8.4 (Pin_4)
- net OLED_SCL: now also J7.4 (Pin_4)
- net OLED_SDA: now also J7.6 (Pin_6)
- net PA0: now also J9.3 (Pin_3)
- net PB0: now also J9.4 (Pin_4)
- net PB1: now also J9.5 (Pin_5)
- net PB3: now also J9.6 (Pin_6)
- net PB4: now also J9.7 (Pin_7)
- net PB5: now also J9.8 (Pin_8)
- net PC13: now also J9.9 (Pin_9)
- net PC14: now also J9.10 (Pin_10)
- net PC15: now also J9.11 (Pin_11)
- net SPI1_MISO: now also J7.5 (Pin_5)
- net SPI1_NSS: now also J7.3 (Pin_3)
