File: InitialDesign/Power.sch (KiCad schematic (older format))
At the start: 7 parts, among them U1 TPS61222DCKR

Commit message: Schematic and Layout commenced
Parts:
- BT1: footprint (none) -> Battery_Holders:Keystone_2466_1xAAA
- C1, C2: footprint (none) -> Capacitors_SMD:CP_Elec_4x5.3
- L1: footprint (none) -> Inductors_SMD:L_Taiyo-Yuden_NR-30xx
- R3, R4: footprint (none) -> Resistors_SMD:R_0805
- U1: footprint (none) -> lib_dp:SC-70-6
Changed lines of the file:
@@
 F 0 "U1" H 5650 4500 60  0000 C CNN
 F 1 "TPS61222DCKR" H 5850 3800 60  0000 C CNN
-F 2 "" H 5600 3950 60  0001 C CNN
+F 2 "lib_dp:SC-70-6" H 5600 3950 60  0001 C CNN
 F 3 "" H 5600 3950 60  0001 C CNN
 	1    5850 4200
@@
 F 0 "L1" V 5100 4000 50  0000 C CNN
 F 1 "4.7uH" V 5225 4000 50  0000 C CNN
-F 2 "" H 5150 4000 50  0001 C CNN
+F 2 "Inductors_SMD:L_Taiyo-Yuden_NR-30xx" H 5150 4000 50  0001 C CNN
 F 3 "" H 5150 4000 50  0001 C CNN
 	1    5150 4000
@@
 F 0 "C1" H 5025 4400 50  0000 L CNN
 F 1 "10uF" H 5025 4200 50  0000 L CNN
-F 2 "" H 5038 4150 50  0001 C CNN
+F 2 "Capacitors_SMD:CP_Elec_4x5.3" H 5038 4150 50  0001 C CNN
 F 3 "" H 5000 4300 50  0001 C CNN
 	1    5000 4300
@@
 F 0 "C2" H 6725 4250 50  0000 L CNN
 F 1 "10uF" H 6725 4050 50  0000 L CNN
-F 2 "" H 6738 4000 50  0001 C CNN
+F 2 "Capacitors_SMD:CP_Elec_4x5.3" H 6738 4000 50  0001 C CNN
 F 3 "" H 6700 4150 50  0001 C CNN
 	1    6700 4150
@@
 F 0 "R3" V 6480 4200 50  0000 C CNN
 F 1 "2.7M" V 6400 4200 50  0000 C CNN
-F 2 "" V 6330 4200 50  0001 C CNN
+F 2 "Resistors_SMD:R_0805" V 6330 4200 50  0001 C CNN
 F 3 "" H 6400 4200 50  0001 C CNN
 	1    6400 4200
@@
 F 0 "R4" V 6480 4550 50  0000 C CNN
 F 1 "470k" V 6400 4550 50  0000 C CNN
-F 2 "" V 6330 4550 50  0001 C CNN
+F 2 "Resistors_SMD:R_0805" V 6330 4550 50  0001 C CNN
 F 3 "" H 6400 4550 50  0001 C CNN
 	1    6400 4550
@@
 	6700 4000 6250 4000
 $Comp
-L GND #PWR011
+L GND #PWR013
 U 1 1 5A51E15C
 P 5400 4750
-F 0 "#PWR011" H 5400 4500 50  0001 C CNN
+F 0 "#PWR013" H 5400 4500 50  0001 C CNN
 F 1 "GND" H 5400 4600 50  0000 C CNN
 F 2 "" H 5400 4750 50  0001 C CNN
@@
 	5400 4400 5400 4750
 $Comp
-L GND #PWR012
+L GND #PWR014
 U 1 1 5A51E1A7
 P 6400 4750
-F 0 "#PWR012" H 6400 4500 50  0001 C CNN
+F 0 "#PWR014" H 6400 4500 50  0001 C CNN
 F 1 "GND" H 6400 4600 50  0000 C CNN
 F 2 "" H 6400 4750 50  0001 C CNN
@@
 	6400 4750 6400 4700
 $Comp
-L GND #PWR013
+L GND #PWR015
 U 1 1 5A51E1DA
 P 6700 4300
-F 0 "#PWR013" H 6700 4050 50  0001 C CNN
+F 0 "#PWR015" H 6700 4050 50  0001 C CNN
 F 1 "GND" H 6700 4150 50  0000 C CNN
 F 2 "" H 6700 4300 50  0001 C CNN
@@
 F 0 "BT1" H 4450 4400 50  0000 R CNN
 F 1 "1020_Keystone" H 4450 4300 50  0000 R CNN
-F 2 "" V 4600 4360 50  0001 C CNN
+F 2 "Battery_Holders:Keystone_2466_1xAAA" V 4600 4360 50  0001 C CNN
 F 3 "" V 4600 4360 50  0001 C CNN
 	1    4600 4300
@@
 	4600 4400 4600 4450
 $Comp
-L +3V3 #PWR014
+L +3V3 #PWR016
 U 1 1 5A51E6C2
 P 6700 3850
-F 0 "#PWR014" H 6700 3700 50  0001 C CNN
+F 0 "#PWR016" H 6700 3700 50  0001 C CNN
 F 1 "+3V3" H 6700 3990 50  0000 C CNN
 F 2 "" H 6700 3850 50  0001 C CNN
@@
 	6700 3850 6700 4000
 $Comp
-L +BATT #PWR015
+L +BATT #PWR017
 U 1 1 5A54DBA7
 P 4600 3950
-F 0 "#PWR015" H 4600 3800 50  0001 C CNN
+F 0 "#PWR017" H 4600 3800 50  0001 C CNN
 F 1 "+BATT" H 4600 4090 50  0000 C CNN
 F 2 "" H 4600 3950 50  0001 C CNN
@@
 Wire Wire Line
 	6400 4400 6400 4350
+Connection ~ 5400 4450
 $EndSCHEMATC
